Commit message: change base frame of stl

File: sun_tactile_simulation/urdf/sun_finger_v3.xacro (robot description, xacro)
@@ -18,5 +18,5 @@
 </xacro:property>
 <xacro:property name="mesh_origin">
-  <origin xyz="${-56.9550247192*local_scale} ${-45.514275551*local_scale} ${0.00445556640625*local_scale}" rpy="${pi/2.0} ${0.0} ${pi/2}" />
+  <!--origin xyz="${-56.9550247192*local_scale} ${-45.514275551*local_scale} ${0.00445556640625*local_scale}" rpy="${pi/2.0} ${0.0} ${pi/2}" /-->
 </xacro:property>
 <link name="${link_name}">

Commit message: Add color

File: sun_tactile_simulation/urdf/sun_finger_v3.xacro (robot description, xacro)
@@ -26,4 +26,7 @@
             <xacro:insert_block name="finger_mesh" />
         </geometry>
+        <material name="blue">
+            <color rgba="0 0 0.8 1"/>
+        </material>
     </visual>
     <collision>
