Commit message: tf_prefix in nodes

File: sun_tactile_simulation/urdf/wsg50_with_sunfinger.xacro (robot description, xacro)
@@ -12,6 +12,7 @@
     create_sensor_link = if true create a link for the sensor frame (default true)
                          the sensor frame will be ${prefix}(left|right)/sensor_frame
-    create_sensor_link = if true create a link for the grasp frame (default true)
+    create_grasp_link = if true create a link for the grasp frame (default true)
                          the grasp frame will be ${prefix}/grasp_frame
+    rotate_grasp_link = if true rotate the grasp link of 180° about x axis (default false)
     the gripper base link will be ${prefix}${base_link}
     the two prismatic joints : ${prefix}left/finger_flange_joint and ${prefix}right/finger_flange_joint
@@ -28,4 +29,5 @@
         create_sensor_link:=true
         create_grasp_link:=true
+        rotate_grasp_link:=false
         "
 >
@@ -99,4 +101,8 @@
     />
     <!-- grasp frame -->
+    <xacro:property name="delta_rpy_y" value="0"/>
+    <xacro:if value="${rotate_grasp_link}">
+        <xacro:property name="delta_rpy_y" value="${pi}"/>
+    </xacro:if>
     <xacro:if value="${create_grasp_link}">
         <link name="${prefix}grasp_frame" />
@@ -104,5 +110,5 @@
             <parent link="${prefix}${base_link}" />
             <child link="${prefix}grasp_frame" />
-            <origin xyz="0 0 ${0.191486403*scale}" rpy="${pi/2} 0 ${pi/2}" />
+            <origin xyz="0 0 ${0.191486403*scale}" rpy="${pi/2} 0 ${pi/2+delta_rpy_y}" />
         </joint>
     </xacro:if>
