Commit message: Finger v3N for wsg50

File: sun_tactile_simulation/urdf/wsg50_with_sunfinger.urdf.xacro (robot description, xacro)
@@ -7,5 +7,5 @@
     base_link="base_link"
     scale="1.0"
-    finger_version="v3"
+    finger_version="v3N"
     mimic_joints="true"
     create_sensor_link="true"

File: sun_tactile_simulation/urdf/wsg50_with_sunfinger.xacro (robot description, xacro)
@@ -39,4 +39,10 @@
     <xacro:property name="finger_flange_right_link" value="${finger_flange_link}"/>
     <xacro:property name="sun_finger_link" value="sun_finger_link"/>
+    <xacro:if value="${finger_version=='v3'}">
+        <xacro:property name="grasp_dz" value="0.191486403"/>
+    </xacro:if>
+    <xacro:if value="${finger_version=='v3N'}">
+        <xacro:property name="grasp_dz" value="0.1830145968018"/>
+    </xacro:if>
     <!-- wsg50 without fingers -->
     <!--
@@ -87,4 +93,15 @@
             />
         </xacro:if>
+        <!-- Finger V3N -->
+        <xacro:if value="${finger_version=='v3N'}">
+            <!-- Import finger macro -->
+            <xacro:include filename="$(find sun_tactile_simulation)/urdf/sun_finger_v3N.xacro" />
+            <xacro:sun_finger_v3N
+                scale="${scale}"
+                base_link="${finger_link}"
+                prefix="${prefix}"
+                create_sensor_link="${create_sensor_link}"
+            />
+        </xacro:if>
     </xacro:macro> <!-- end macro sun_finger_with_fixed_joint -->
     <xacro:sun_finger_with_fixed_joint
@@ -110,5 +127,5 @@
             <parent link="${prefix}${base_link}" />
             <child link="${prefix}grasp_frame" />
-            <origin xyz="0 0 ${0.191486403*scale}" rpy="${pi/2} 0 ${pi/2+delta_rpy_y}" />
+            <origin xyz="0 0 ${grasp_dz*scale}" rpy="${pi/2} 0 ${pi/2+delta_rpy_y}" />
         </joint>
     </xacro:if>

Commit message: add finger v4

File: sun_tactile_simulation/urdf/wsg50_with_sunfinger.urdf.xacro (robot description, xacro)
@@ -1,4 +1,4 @@
 <?xml version="1.0"?>
-<robot name="sun_finger_v3" xmlns:xacro="http://www.ros.org/wiki/xacro">
+<robot name="sun_finger_v4" xmlns:xacro="http://www.ros.org/wiki/xacro">
   <!-- Import finger macro -->
   <xacro:include filename="$(find sun_tactile_simulation)/urdf/wsg50_with_sunfinger.xacro" />
@@ -7,5 +7,5 @@
     base_link="base_link"
     scale="1.0"
-    finger_version="v3N"
+    finger_version="v4"
     mimic_joints="true"
     create_sensor_link="true"

File: sun_tactile_simulation/urdf/wsg50_with_sunfinger.xacro (robot description, xacro)
@@ -25,5 +25,5 @@
         base_link:=base_link
         scale:=1.0
-        finger_version:=v3
+        finger_version:=v4
         mimic_joints:=true
         create_sensor_link:=true
@@ -44,4 +44,7 @@
     <xacro:if value="${finger_version=='v3N'}">
         <xacro:property name="grasp_dz" value="0.1830145968018"/>
+    </xacro:if>
+    <xacro:if value="${finger_version=='v4'}">
+        <xacro:property name="grasp_dz" value="0.183356"/>
     </xacro:if>
     <!-- wsg50 without fingers -->
@@ -104,4 +107,15 @@
             />
         </xacro:if>
+        <!-- Finger V4 -->
+        <xacro:if value="${finger_version=='v4'}">
+            <!-- Import finger macro -->
+            <xacro:include filename="$(find sun_tactile_simulation)/urdf/sun_finger_v4.xacro" />
+            <xacro:sun_finger_v4
+                scale="${scale}"
+                base_link="${finger_link}"
+                prefix="${prefix}"
+                create_sensor_link="${create_sensor_link}"
+            />
+        </xacro:if>
     </xacro:macro> <!-- end macro sun_finger_with_fixed_joint -->
     <xacro:sun_finger_with_fixed_joint
@@ -130,4 +144,4 @@
         </joint>
     </xacro:if>
-</xacro:macro> <!-- end wsg50_with_fingerv3 -->
+</xacro:macro> <!-- end wsg50_with_finger -->
 </robot>
